File: electronics/reset_switch/reset_switch.sch (KiCad schematic (older format))
At the start: 7 parts, among them P1 CONN_01X04, Q1 Fairchild_BCV27, Q2 QRE1113

Commit message: Smaller mount holes, fixed R2 R3 labels. Cleaner Q2 to show pin 1
Parts:
- Q2: footprint SparkFun:SparkFun-QRE1113 -> custom_footprints:SparkFun-QRE1113
Changed lines of the file:
@@
 F 0 "Q2" H 5400 3450 50  0000 C CNN
 F 1 "QRE1113" H 5750 3050 50  0000 C CNN
-F 2 "SparkFun:SparkFun-QRE1113" H 5350 3300 60  0001 C CNN
+F 2 "custom_footprints:SparkFun-QRE1113" H 5350 3300 60  0001 C CNN
 F 3 "" H 5350 3300 60  0000 C CNN
 	1    5350 3300
